File: hardware/hardware.kicad_sch (KiCad schematic)
At the start: 5 parts, among them J2 RFShield_OnePiece

Commit message: Added hardware SDI-12
Parts:
- J2: MFC (none) -> Würth Elektronik; MPN (none) -> 36103305S,36003300S
Changed lines of the file:
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@@
+      (effects (font (size 1.27 1.27)) hide)
+    )
+    (property "MPN" "36103305S,36003300S" (at 62.23 46.99 0)
+      (effects (font (size 1.27 1.27)) hide)
+    )
+    (property "MFC" "Würth Elektronik" (at 62.23 46.99 0)
       (effects (font (size 1.27 1.27)) hide)
     )

Commit message: Updated annotations based on PCB position
Other:
- company: (none) -> jlab
- title: (none) -> Soil Power Sensor
Changed lines of the file:
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@@
 (kicad_sch (version 20230121) (generator eeschema)
   (paper "A4")
+  (title_block
+    (title "Soil Power Sensor")
+    (date "2024-03-08")
+    (rev "2.2.0")
+    (company "jlab")
+  )
   (rectangle (start 25.4 20.32) (end 101.6 66.04)
     (stroke (width 0) (type default))

Commit message: Generated BOM
Parts:
- added J6: RFShield_OnePiece, symbol Device:RFShield_OnePiece
- J2: MPN 36103305S,36003300S -> 36103305S
Connections:
- net GND: now also J6.1 (Shield)
Other:
- note added: "Cover not placed"
- note added: "Frame placed on PCB"
Changed lines of the file:
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@@
     (company "jlab")
   )
-  (rectangle (start 25.4 20.32) (end 101.6 66.04)
+  (rectangle (start 25.4 20.32) (end 101.6 106.68)
     (stroke (width 0) (type default))
     (fill (type none))
@@
   (text "RF Shield" (at 26.67 25.4 0)
     (effects (font (size 2.54 2.54)) (justify left bottom))
+  )
+  (text "Frame placed\non PCB" (at 30.48 46.99 0)
+    (effects (font (size 1.27 1.27)) (justify left bottom))
+  )
+  (text "Cover not placed" (at 27.94 80.01 0)
+    (effects (font (size 1.27 1.27)) (justify left bottom))
   )
   (symbol (lib_id "Mechanical:MountingHole_Pad") (at 128.27 52.07 0) (unit 1)
@@
       (effects (font (size 1.27 1.27)) hide)
     )
-    (property "MPN" "36103305S,36003300S" (at 62.23 46.99 0)
+    (property "MPN" "36103305S" (at 62.23 46.99 0)
       (effects (font (size 1.27 1.27)) hide)
     )
@@
         (path "/5300ec4d-4648-40a1-8d89-4fa6b3bf32a3/e8086a96-0786-4ae2-b425-e1003c006b3a"
           (reference "J2") (unit 1)
+        )
+      )
+    )
+  )
+  (symbol (lib_id "power:GND") (at 62.23 90.17 0) (unit 1)
+    (in_bom yes) (on_board yes) (dnp no) (fields_autoplaced)
+    (property "Reference" "#PWR017" (at 62.23 96.52 0)
+      (effects (font (size 1.27 1.27)) hide)
+    )
+    (property "Value" "GND" (at 62.23 95.25 0)
+      (effects (font (size 1.27 1.27)))
+    )
+    (property "Footprint" "" (at 62.23 90.17 0)
+      (effects (font (size 1.27 1.27)) hide)
+    )
+    (property "Datasheet" "" (at 62.23 90.17 0)
+      (effects (font (size 1.27 1.27)) hide)
+    )
+    (pin "1")
+    (instances
+      (project "Soil Power Sensor"
+        (path "/5300ec4d-4648-40a1-8d89-4fa6b3bf32a3/e8086a96-0786-4ae2-b425-e1003c006b3a"
+          (reference "#PWR017") (unit 1)
         )
       )
@@
         )
       )
+    )
+  )
+  (symbol (lib_id "Device:RFShield_OnePiece") (at 62.23 80.01 0) (unit 1)
+    (in_bom yes) (on_board yes) (dnp no)
+    (property "Reference" "J6" (at 46.99 67.31 0)
+      (effects (font (size 1.27 1.27)) (justify left))
+    )
+    (property "Value" "RFShield_OnePiece" (at 46.99 69.85 0)
+      (effects (font (size 1.27 1.27)) (justify left))
+    )
+    (property "Footprint" "" (at 62.23 82.55 0)
+      (effects (font (size 1.27 1.27)) hide)
+    )
+    (property "Datasheet" "~" (at 62.23 82.55 0)
+      (effects (font (size 1.27 1.27)) hide)
+    )
+    (property "MPN" "36003300S" (at 62.23 80.01 0)
+      (effects (font (size 1.27 1.27)) hide)
+    )
+    (property "MFC" "Würth Elektronik" (at 62.23 80.01 0)
+      (effects (font (size 1.27 1.27)) hide)
+    )
+    (pin "1")
+    (instances
+      (project "Soil Power Sensor"
+        (path "/5300ec4d-4648-40a1-8d89-4fa6b3bf32a3/e8086a96-0786-4ae2-b425-e1003c006b3a"
+          (reference "J6") (unit 1)
+        )
+      )
