File: hardware/Soil Power Sensor.kicad_pcb (KiCad board)
At the start: 2 copper layers, 139 x 45 mm, 67 parts, among them J1 Screw_Terminal_01x05, J2 RFShield_OnePiece, J3 UART, J4 Conn_01x03, J5 Micro_SD_Card, J7 Conn_01x04_Socket, Q1 BSS123, SW1 BOOT, SW2 EN, U1 MAX9944, U10 Wio-E5 mini, U11 MB85RC1MT, U12 MB85RC1MT, U2 INA296A, U3 REF2033, U4 THS4532, U5 TPS60400DBV, U6 ADS1219, U7 SN74LVC1G240, U8 ESP32-C3-WROOM-02-N4

Commit message: Closes #60
Parts:
- R18: renamed from RSENSE1; value DNP -> 2.2k; footprint Resistor_SMD:R_0603_1608Metric -> Capacitor_SMD:C_0603_1608Metric
- turned R18 to -90 degrees
Connections:
- R18 pad 1: Net-(JP1-A) -> /Analog/I-
- R18 pad 2: /Analog/I- -> Net-(JP1-A)
Changed lines of the file:
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@@
 		)
 	)
-	(footprint "Resistor_SMD:R_0603_1608Metric"
+	(footprint "Capacitor_SMD:C_0603_1608Metric"
 		(layer "F.Cu")
-		(at 128.5 65 90)
-		(descr "Resistor SMD 0603 (1608 Metric), square (rectangular) end terminal, IPC_7351 nominal, (Body size source: IPC-SM-782 page 72, https://www.pcb-3d.com/wordpress/wp-content/uploads/ipc-sm-782a_amendment_1_and_2.pdf), generated with kicad-footprint-generator")
-		(tags "resistor")
-		(property "Reference" "RSENSE1"
-			(at 2.5 0 180)
+		(at 128.5 65 -90)
+		(descr "Capacitor SMD 0603 (1608 Metric), square (rectangular) end terminal, IPC_7351 nominal, (Body size source: IPC-SM-782 page 76, https://www.pcb-3d.com/wordpress/wp-content/uploads/ipc-sm-782a_amendment_1_and_2.pdf), generated with kicad-footprint-generator")
+		(tags "capacitor")
+		(property "Reference" "R18"
+			(at -2 0.1 360)
 			(layer "F.SilkS")
-			(hide yes)
 			(effects
 				(font
@@
 			)
 		)
-		(property "Value" "DNP"
-			(at 2.505 0 90)
+		(property "Value" "2.2k"
+			(at 2 -0.1 360)
 			(layer "F.Fab")
-			(hide yes)
 			(effects
 				(font
@@
 			)
 		)
-		(property "Footprint" "Resistor_SMD:R_0603_1608Metric"
-			(at 0 0 90)
+		(property "Footprint" "Capacitor_SMD:C_0603_1608Metric"
+			(at 0 0 -90)
 			(unlocked yes)
 			(layer "F.Fab")
@@
 		)
 		(property "Datasheet" ""
-			(at 0 0 90)
+			(at 0 0 -90)
 			(unlocked yes)
 			(layer "F.Fab")
@@
 		)
 		(property "Description" "Resistor"
-			(at 0 0 90)
+			(at 0 0 -90)
 			(unlocked yes)
 			(layer "F.Fab")
@@
 			)
 		)
-		(property "LCSC" ""
-			(at 0 0 90)
-			(unlocked yes)
-			(layer "F.Fab")
-			(hide yes)
-			(effects
-				(font
-					(size 1 1)
-					(thickness 0.15)
-				)
-			)
-		)
 		(property ki_fp_filters "R_*")
 		(sheetname "Analog")
 		(sheetfile "Soil_Power_Sensor_1.kicad_sch")
-		(attr smd exclude_from_bom dnp)
+		(attr smd)
 		(fp_line
-			(start -0.237258 -0.5225)
-			(end 0.237258 -0.5225)
+			(start -0.14058 0.51)
+			(end 0.14058 0.51)
 			(stroke
 				(width 0.12)
@@
 		)
 		(fp_line
-			(start -0.237258 0.5225)
-			(end 0.237258 0.5225)
+			(start -0.14058 -0.51)
+			(end 0.14058 -0.51)
 			(stroke
 				(width 0.12)
@@
 		)
 		(fp_line
-			(start 1.48 -0.73)
-			(end 1.48 0.73)
+			(start -1.48 0.73)
+			(end -1.48 -0.73)
+			(stroke
+				(width 0.05)
+				(type solid)
+			)
+			(layer "F.CrtYd")
+		)
+		(fp_line
+			(start 1.48 0.73)
+			(end -1.48 0.73)
 			(stroke
 				(width 0.05)
@@
 		)
 		(fp_line
-			(start 1.48 0.73)
-			(end -1.48 0.73)
+			(start 1.48 -0.73)
+			(end 1.48 0.73)
 			(stroke
 				(width 0.05)
@@
 		)
 		(fp_line
-			(start -1.48 0.73)
-			(end -1.48 -0.73)
-			(stroke
-				(width 0.05)
-				(type solid)
-			)
-			(layer "F.CrtYd")
-		)
-		(fp_line
-			(start 0.8 -0.4125)
-			(end 0.8 0.4125)
+			(start -0.8 0.4)
+			(end -0.8 -0.4)
 			(stroke
 				(width 0.1)
@@
 		)
 		(fp_line
-			(start -0.8 -0.4125)
-			(end 0.8 -0.4125)
+			(start 0.8 0.4)
+			(end -0.8 0.4)
 			(stroke
 				(width 0.1)
@@
 		)
 		(fp_line
-			(start 0.8 0.4125)
-			(end -0.8 0.4125)
+			(start -0.8 -0.4)
+			(end 0.8 -0.4)
 			(stroke
 				(width 0.1)
@@
 		)
 		(fp_line
-			(start -0.8 0.4125)
-			(end -0.8 -0.4125)
+			(start 0.8 -0.4)
+			(end 0.8 0.4)
 			(stroke
 				(width 0.1)
@@
 		)
 		(pad "1" smd roundrect
-			(at -0.825 0 90)
-			(size 0.8 0.95)
+			(at -0.775 0 270)
+			(size 0.9 0.95)
+			(layers "F.Cu" "F.Paste" "F.Mask")
+			(roundrect_rratio 0.25)
+			(net 25 "/Analog/I-")
+			(pintype "passive")
+		)
+		(pad "2" smd roundrect
+			(at 0.775 0 270)
+			(size 0.9 0.95)
 			(layers "F.Cu" "F.Paste" "F.Mask")
 			(roundrect_rratio 0.25)
@@
 			(pintype "passive")
 		)
-		(pad "2" smd roundrect
-			(at 0.825 0 90)
-			(size 0.8 0.95)
-			(layers "F.Cu" "F.Paste" "F.Mask")
-			(roundrect_rratio 0.25)
-			(net 25 "/Analog/I-")
-			(pintype "passive")
-		)
-		(model "${KICAD8_3DMODEL_DIR}/Resistor_SMD.3dshapes/R_0603_1608Metric.wrl"
+		(model "${KICAD8_3DMODEL_DIR}/Capacitor_SMD.3dshapes/C_0603_1608Metric.wrl"
 			(offset
 				(xyz 0 0 0)

Commit message: Routed PCB
Parts:
- removed TP3: +3V3, TestPoint:TestPoint_Pad_D1.5mm
- added J8: Conn_01x10, Connector_PinHeader_2.54mm:PinHeader_1x10_P2.54mm_Horizontal, F.Cu at (246.4, 58.1)
- added Q2: L8050QLT1G, Package_TO_SOT_SMD:SOT-23, F.Cu at (161.6, 88.8)
- added Q3: L8050QLT1G, Package_TO_SOT_SMD:SOT-23, F.Cu at (154.6, 84.8)
- added R19: 10k, Resistor_SMD:R_0603_1608Metric, F.Cu at (154.7, 89.8)
- added R20: 10k, Resistor_SMD:R_0603_1608Metric, F.Cu at (161.5, 83.8)
- added TP5: VCC, TestPoint:TestPoint_Pad_3.0x3.0mm, F.Cu at (213.2, 50.6)
- J3: value UART -> Debug; footprint Connector_PinHeader_2.54mm:PinHeader_1x04_P2.54mm_Vertical -> Connector_PinHeader_2.54mm:PinHeader_2x05_P2.54mm_Vertical
- moved R17 40.6 mm to (213.9, 59.1), turned to 0 degrees
- moved R16 39.6 mm to (213.8, 55.6), turned to 180 degrees
- moved R12 13.0 mm to (170.8, 76.0)
- moved TP4 12.9 mm to (147.2, 86.2)
- moved TP1 5.64 mm to (128.0, 86.2)
- moved TP2 4.19 mm to (138.5, 86.2)
- moved J3 2.26 mm to (169.1, 79.1)
- moved U8 1.95 mm to (186.2, 88.1)
- moved J5 1.20 mm to (205.0, 84.6)
- moved JP2 0.50 mm to (128.5, 60.0)
Connections:
- J3 pad 1: VCC -> /ESP32/DTR
- J3 pad 2: /ESP32/RX -> /ESP32/USB_D+
- J3 pad 3: /ESP32/TX -> /ESP32/RTS
- J3 pad 4: GND -> /ESP32/USB_D-
- U10 pad 24: VUSB -> VCC
- U8 pad 13: unconnected-(U8-IO18-Pad13) -> /ESP32/USB_D-
- U8 pad 14: unconnected-(U8-IO19-Pad14) -> /ESP32/USB_D+
Routing:
- net (no net): track 280.2 -> 0.00 mm, vias 1 -> 0
- net +3V3: track 321.8 -> 252.4 mm, vias 15 -> 18
- net Net-(U10-SCK/PB13): track 10.6 -> 65.3 mm
- net VCC: track 214.0 -> 169.5 mm, vias 3 -> 2
- net /ESP32/EN: track 36.8 -> 72.3 mm, vias 0 -> 2
- net /ESP32/BOOT: track 25.1 -> 59.8 mm, vias 0 -> 2
- net VUSB: track 28.0 -> 0.00 mm, vias 1 -> 0
- net /ESP32/DTR: track 0.00 -> 23.9 mm
- net /Analog/POWERDOWN: track 153.5 -> 134.0 mm
- net /ESP32/RTS: track 0.00 -> 16.2 mm
- net GND: track 142.5 -> 128.5 mm, vias 23 -> 26
- net Net-(U8-IO2): track 5.09 -> 15.7 mm, vias 0 -> 2
- net /ESP32/USB_D+: track 0.00 -> 9.80 mm, vias 0 -> 1
- net /ESP32/RX: track 5.90 -> 15.4 mm
- net Net-(Q3-B): track 0.00 -> 7.86 mm
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Other:
- board text added: "D+"
- board text added: "D-"
- board text added: "DTR"
- board text added: "RTS"
- board text removed: "+3V3"
- board text removed: "BAT"
- board text removed: "USB"
- board text removed: "VBAT"
- board text removed: "VUSB"
