File: hardware/Soil Power Sensor.kicad_pcb (KiCad board)
At the start: 2 copper layers, 151 x 103.2 mm, 138 parts, among them J1 Conn_01x02, J10 Conn_01x04_Socket, J11 Conn_01x04_Pin, J12 Conn_01x04_Socket, J13 USB_C_Receptacle_USB2.0_16P, J15 Conn_01x03, J16 Micro_SD_Card, J2 DC050-T, J3 Conn_01x10_Pin, J4 Conn_01x03, J5 AudioJack3, J6 SMA-K, J7 U-FL, J8 Conn_01x03, J9 Conn_01x06_Pin, Q1 BSS123, Q10 AO3401A, Q2 AO3401A, Q3 AO3401A, Q6 AO3401A, Q7 AO3401A, Q8 AO3401A, Q9 BSS123, SW3 RST, SW4 BOOT/USER, SW5 BOOT, SW6 EN, U1 BQ24210DQCR, U10 TCA9535PWR, U11 TPS631000DRLR, U3 SN74LVC1G240, U4 LoRa-E5, U5 MB85RC1MT, U6 MAX3072E, U7 MB85RC1MT, U8 CP2102N-Axx-xQFN24, U9 ESP32-C3-WROOM-02-N4

Commit message: rough layout spacing
Parts:
- removed D10: LED, LED_SMD:LED_0603_1608Metric
- removed D11, D12: D, Diode_SMD:D_0603_1608Metric
- removed F2: Fuse_Small, Fuse:Fuse_0603_1608Metric
- removed F3: Polyfuse, Fuse:Fuse_0603_1608Metric
- removed Q10: AO3401A, Package_TO_SOT_SMD:SOT-23
- removed Q9: BSS123, Package_TO_SOT_SMD:SOT-23
- removed RT1: 21.5 kOhm, Resistor_SMD:R_0603_1608Metric
- removed SW5: BOOT, Button_Switch_SMD:SW_Push_1P1T_NO_CK_KSC7xxJ
- removed SW6: EN, Button_Switch_SMD:SW_Push_1P1T_NO_CK_KSC7xxJ
- removed U3: SN74LVC1G240, Package_TO_SOT_SMD:SOT-23-5
- added BT1: Battery_Cell, Connector_JST:JST_PH_S2B-PH-K_1x02_P2.00mm_Horizontal, F.Cu at (72.5, -11.8)
- added F1: Fuse_Small, Fuse:Fuse_0603_1608Metric, F.Cu at (-52.5, 134.0)
- added J14: USB_C_Receptacle_USB2.0_16P, Connector_USB:USB_C_Receptacle_GCT_USB4110, F.Cu at (-50.0, 141.0)
- added J17: Conn_01x03, Connector_PinHeader_2.54mm:PinHeader_1x03_P2.54mm_Vertical, F.Cu at (276.0, -75.0)
- added J18: Conn_01x03, Connector_PinHeader_2.54mm:PinHeader_1x03_P2.54mm_Vertical, F.Cu at (272.0, -70.5)
- added J19: Micro_SD_Card, Connector_Card:microSD_HC_Molex_104031-0811, F.Cu at (242.3, -73.8)
- added JP14: SolderJumper_3_Open, Jumper:SolderJumper-3_P1.3mm_Open_Pad1.0x1.5mm, F.Cu at (136.0, 139.5)
- added JP15: SolderJumper_2_Open, Jumper:SolderJumper-2_P1.3mm_Open_RoundedPad1.0x1.5mm, F.Cu at (-17.0, 106.5)
- added JP16: SolderJumper_2_Open, Jumper:SolderJumper-2_P1.3mm_Open_RoundedPad1.0x1.5mm, F.Cu at (-14.0, 104.0)
- added JP17: SolderJumper_2_Open, Jumper:SolderJumper-2_P1.3mm_Open_RoundedPad1.0x1.5mm, F.Cu at (-17.0, 103.0)
- added JP18: SolderJumper_2_Open, Jumper:SolderJumper-2_P1.3mm_Open_RoundedPad1.0x1.5mm, F.Cu at (-14.0, 101.5)
- added JP19: SolderJumper_2_Open, Jumper:SolderJumper-2_P1.3mm_Open_RoundedPad1.0x1.5mm, F.Cu at (-17.0, 99.5)
- added Q4: AO3400A, Package_TO_SOT_SMD:SOT-23, F.Cu at (406.5, 219.5)
- added Q5: AO3401A, Package_TO_SOT_SMD:SOT-23, F.Cu at (366.4, 130.1)
- added R25: 47k, Resistor_SMD:R_0603_1608Metric, F.Cu at (365.7, 144.0)
- added R32: 20, Resistor_SMD:R_0603_1608Metric, F.Cu at (-55.0, 121.0)
- added R33: 1k, Resistor_SMD:R_0603_1608Metric, F.Cu at (-46.0, 123.8)
- added R46: 22.1k, Resistor_SMD:R_0603_1608Metric, F.Cu at (-52.5, 128.0)
- added R47: 47.5k, Resistor_SMD:R_0603_1608Metric, F.Cu at (-52.5, 126.5)
- added SW1: RST, Button_Switch_SMD:SW_Push_1P1T_NO_CK_KSC7xxJ, F.Cu at (108.9, 81.5)
- added SW2: BOOT/USER, Button_Switch_SMD:SW_Push_1P1T_NO_CK_KSC7xxJ, F.Cu at (92.6, 81.5)
- added U2: TPS63900, Package_SON:WSON-10-1EP_2.5x2.5mm_P0.5mm_EP1.2x2mm_ThermalVias, F.Cu at (104.5, -11.8)
- C1, C2: value 1 uF -> 1uF
- C10, C13, C3: value 100nF -> 0.1uF
- C11, C12, C19, C6: value 10uF -> 0.1uF
- C16: value 1uF -> 0.1uF
- C17, C9: value 0.1uF -> 10uF
- C20: value 0.1uF -> 1uF
- C21: value 47 uF -> 0.1uF
- C5: value 100nF -> 47uF
- C7: value 47 uF -> 10uF
- C8: value 0.1uF -> 47uF
- D1, D2: value LED -> RB521S-40; footprint LED_SMD:LED_0603_1608Metric -> Diode_SMD:D_SOD-523
- D4: value ARM10_DEBUG -> LED; footprint Soil Power Sensor:ARM10_DEBUG -> LED_SMD:LED_0603_1608Metric
- D6, D8: value ESD131-B1-W0201 -> LED; footprint Diode_SMD:Infineon_SG-WLL-2-3_0.58x0.28_P0.36mm -> LED_SMD:LED_0603_1608Metric
- D7: value ESD131-B1-W0201 -> SP0503BAHT; footprint Diode_SMD:Infineon_SG-WLL-2-3_0.58x0.28_P0.36mm -> Package_TO_SOT_SMD:SOT-143
- FL1: value 0603USB-222 -> SRF2012-900YA; footprint Inductor_SMD:L_CommonModeChoke_Coilcraft_0603USB -> Soil Power Sensor:IND_BOURNS_SRF2012A
- J1: value Conn_01x02 -> DC050-T; footprint Connector_JST:JST_PH_S2B-PH-K_1x02_P2.00mm_Horizontal -> Connector_BarrelJack:BarrelJack_Horizontal
- J10: value Conn_01x04_Socket -> Conn_01x03; footprint Connector_JST:JST_SH_SM04B-SRSS-TB_1x04-1MP_P1.00mm_Horizontal -> TerminalBlock_Phoenix:TerminalBlock_Phoenix_PT-1,5-3-5.0-H_1x03_P5.00mm_Horizontal
- J11: footprint Connector_PinHeader_2.54mm:PinHeader_1x04_P2.54mm_Vertical -> Connector_PinSocket_2.54mm:PinSocket_1x04_P2.54mm_Vertical
- J12: value Conn_01x04_Socket -> Conn_01x04_Pin; footprint Connector_JST:JST_SH_SM04B-SRSS-TB_1x04-1MP_P1.00mm_Horizontal -> Connector_PinSocket_2.54mm:PinSocket_1x04_P2.54mm_Vertical
- J13: value USB_C_Receptacle_USB2.0_16P -> Conn_02x20_Top_Bottom; footprint Connector_USB:USB_C_Receptacle_GCT_USB4110 -> Connector_PinSocket_2.54mm:PinSocket_2x20_P2.54mm_Vertical
- J15: value Conn_01x03 -> Conn_02x05_Top_Bottom; footprint Connector_PinHeader_2.54mm:PinHeader_1x03_P2.54mm_Vertical -> Connector_PinHeader_2.54mm:PinHeader_2x05_P2.54mm_Vertical
- J16: value Micro_SD_Card -> Conn_01x04_Pin; footprint Connector_Card:microSD_HC_Molex_104031-0811 -> Connector_PinSocket_2.54mm:PinSocket_1x06_P2.54mm_Vertical
- J2: value DC050-T -> Conn_01x03; footprint Connector_BarrelJack:BarrelJack_Horizontal -> TerminalBlock_Phoenix:TerminalBlock_Phoenix_PT-1,5-3-5.0-H_1x03_P5.00mm_Horizontal
- J3: value Conn_01x10_Pin -> ARM10_DEBUG; footprint Connector_PinHeader_2.54mm:PinHeader_1x10_P2.54mm_Vertical -> Soil Power Sensor:ARM10_DEBUG
- J4: value Conn_01x03 -> SMA-K; footprint TerminalBlock_Phoenix:TerminalBlock_Phoenix_PT-1,5-3-5.0-H_1x03_P5.00mm_Horizontal -> Connector_Coaxial:SMA_Molex_73251-1153_EdgeMount_Horizontal
- J6: value SMA-K -> U-FL; footprint Connector_Coaxial:SMA_Molex_73251-1153_EdgeMount_Horizontal -> Connector_Coaxial:U.FL_Hirose_U.FL-R-SMT-1_Vertical
- J7: value U-FL -> Conn_01x04_Socket; footprint Connector_Coaxial:U.FL_Hirose_U.FL-R-SMT-1_Vertical -> Connector_JST:JST_SH_SM04B-SRSS-TB_1x04-1MP_P1.00mm_Horizontal
- J8: value Conn_01x03 -> Conn_01x04_Socket; footprint TerminalBlock_Phoenix:TerminalBlock_Phoenix_PT-1,5-3-5.0-H_1x03_P5.00mm_Horizontal -> Connector_JST:JST_SH_SM04B-SRSS-TB_1x04-1MP_P1.00mm_Horizontal
- JP1: value Jumper_2_Bridged -> SolderJumper_2_Open; footprint Connector_PinHeader_2.54mm:PinHeader_1x02_P2.54mm_Vertical -> Jumper:SolderJumper-2_P1.3mm_Open_RoundedPad1.0x1.5mm
- JP11: value SolderJumper_2_Open -> SolderJumper_3_Open; footprint Jumper:SolderJumper-2_P1.3mm_Open_RoundedPad1.0x1.5mm -> Jumper:SolderJumper-3_P1.3mm_Open_Pad1.0x1.5mm
- JP12, JP8: value Jumper_3_Open -> SolderJumper_2_Open; footprint Connector_PinHeader_2.54mm:PinHeader_1x03_P2.54mm_Vertical -> Jumper:SolderJumper-2_P1.3mm_Open_RoundedPad1.0x1.5mm
- JP13: value Jumper_3_Open -> SolderJumper_2_Bridged; footprint Connector_PinHeader_2.54mm:PinHeader_1x03_P2.54mm_Vertical -> Jumper:SolderJumper-2_P1.3mm_Bridged_RoundedPad1.0x1.5mm
- JP3: value SolderJumper_2_Open -> SolderJumper_3_Open; footprint Jumper:SolderJumper-2_P1.3mm_Open_RoundedPad1.0x1.5mm -> Connector_PinHeader_2.54mm:PinHeader_1x03_P2.54mm_Vertical
- JP4: value SolderJumper_2_Open -> Jumper_2_Bridged; footprint Jumper:SolderJumper-2_P1.3mm_Open_RoundedPad1.0x1.5mm -> Connector_PinHeader_2.54mm:PinHeader_1x02_P2.54mm_Vertical
- JP5: value SolderJumper_2_Bridged -> SolderJumper_2_Open; footprint Jumper:SolderJumper-2_P1.3mm_Bridged_RoundedPad1.0x1.5mm -> Jumper:SolderJumper-2_P1.3mm_Open_RoundedPad1.0x1.5mm
- JP6: value SolderJumper_2_Open -> SolderJumper_2_Bridged; footprint Jumper:SolderJumper-2_P1.3mm_Open_RoundedPad1.0x1.5mm -> Jumper:SolderJumper-2_P1.3mm_Bridged_RoundedPad1.0x1.5mm
- L1: value 1uH -> 2.2uH
- Q1: value BSS123 -> AO3401A
- Q3: value AO3401A -> AO3400A
- R1: value 1M -> 10k
- R10, R11: value 510 -> 1M
- R12: value 47k -> 680
- R13: value 0 -> 7.32k
- R14: value 0 -> 100k
- R15, R16: value 0 -> 4.7k
- R17: value 0 -> 510
- R18: value 1k -> 510
- R19: value 20 -> 47k
- R2: value 1M -> 470k
- R20: value 20 -> 0
- R21, R22: value 5.1k -> 0
- R24: value 1k -> 47k
- R26: value 91k -> 47k
- R27: value 10k -> R; footprint Resistor_SMD:R_0603_1608Metric -> Resistor_THT:R_Axial_DIN0207_L6.3mm_D2.5mm_P10.16mm_Horizontal
- R28, R31, R41, R42, R44: value 10k -> 0
- R3, R4: value 2 kOhm -> 470k
- R30: value 0 -> 20
- R34, R35: value 47k -> 5.1k
- R36, R37: value 47k -> 1k
- R38: value 4.7k -> 47k
- R39: value 4.7k -> 10k
- R40, R43: value 470k -> 10k
- R45: value 470k -> 0
- R5, R6: value 1 MOhm -> 2k
- R7: value 7.32 kOhm -> 470k
- R8: value 680 Ohm -> 36.5k
- R9: value 1k -> 21.5k
- SW3: value RST -> EN
- SW4: value BOOT/USER -> BOOT
- TP1: value Vin -> V_{BUS}
- TP2: value VBAT sense -> V_{BAT}/2
- U1: footprint Soil Power Sensor:LoRa-E5 -> Package_SON:WSON-10-1EP_2x3mm_P0.5mm_EP0.84x2.4mm_ThermalVias
- U10: value TCA9535PWR -> CP2102N-Axx-xQFN24; footprint Package_SO:TSSOP-24_4.4x7.8mm_P0.65mm -> Package_DFN_QFN:QFN-24-1EP_4x4mm_P0.5mm_EP2.6x2.6mm
- U11: value TPS631000DRLR -> ESP32-C3-WROOM-02-N4; footprint Soil Power Sensor:TPS631000DRLR_TEX -> Soil Power Sensor:MODULE_ESP32-C3-WROOM-02-N4
- U4: value LoRa-E5 -> SN74LVC1G240; footprint Soil Power Sensor:LoRa-E5 -> Package_TO_SOT_SMD:SOT-23-5
- U5: value MB85RC1MT -> LoRa-E5; footprint Soil Power Sensor:SOP127P505X155-8N -> Soil Power Sensor:LoRa-E5
- U6: value MAX3072E -> MB85RC1MT; footprint Package_SO:SOIC-8_3.9x4.9mm_P1.27mm -> Soil Power Sensor:SOP127P505X155-8N
- U7: value MB85RC1MT -> SN65HVD11HD; footprint Soil Power Sensor:SOP127P505X155-8N -> Package_SO:SOIC-8_3.9x4.9mm_P1.27mm
- U8: value CP2102N-Axx-xQFN24 -> MB85RC1MT; footprint Package_DFN_QFN:QFN-24-1EP_4x4mm_P0.5mm_EP2.6x2.6mm -> Soil Power Sensor:SOP127P505X155-8N
- U9: value ESP32-C3-WROOM-02-N4 -> TCA9535PWR; footprint Soil Power Sensor:MODULE_ESP32-C3-WROOM-02-N4 -> Package_SO:TSSOP-24_4.4x7.8mm_P0.65mm
- moved D5 409.9 mm to (401.5, 219.5), turned to 90 degrees
- moved JP11 396.3 mm to (385.5, 217.0), turned to -90 degrees
- moved Q6 345.2 mm to (362.1, 142.5)
- moved J12 321.3 mm to (357.0, 141.2)
- moved J11 314.7 mm to (357.0, 129.9)
- moved J8 313.2 mm to (351.5, 143.5), turned to -90 degrees
- moved J2 309.2 mm to (378.5, 207.0), turned to -90 degrees
- moved D7 288.8 mm to (-49.0, 134.5), turned to 0 degrees
- moved FL1 288.6 mm to (-49.5, 131.0)
- moved D8 288.3 mm to (-48.5, 118.0), turned to 90 degrees
- moved D9 278.3 mm to (-47.0, 118.0), turned to 90 degrees
- moved C13 265.4 mm to (-34.8, 128.0), turned to 0 degrees
- moved C14 258.1 mm to (-52.5, 129.5), turned to 180 degrees
- moved C19 257.2 mm to (284.4, -48.5), turned to 90 degrees
- moved C20 256.7 mm to (282.9, -48.5), turned to 90 degrees
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Connections:
- C1 pad 1: Net-(D11-K) -> Net-(D1-K)
- C1 pad 2: 0 -> GND
- C11 pad 1: /Power/VUSB -> Net-(U5-RFIO)
- C12 pad 1: /Power/VUSB -> Net-(C12-Pad1)
- C13 pad 1: Net-(U8-~{DTR}) -> +3V3
- C13 pad 2: /STM32/RST -> GND
- C14 pad 1: +3V3 -> /Power/VUSB
- C15 pad 1: +3V3 -> /Power/VUSB
- C16 pad 1: /ESP32/EN -> Net-(U10-~{DTR})
- C16 pad 2: GND -> /STM32/RST
- C17 pad 1: /ESP32/BOOT -> +3V3
- C18 pad 1: /ESP32/EN -> +3V3
- C19 pad 1: +3V3 -> /ESP32/EN
- C2 pad 1: Net-(JP6-B) -> Net-(BT1-+)
- C2 pad 2: 0 -> GND
- C20 pad 1: +3V3 -> /ESP32/EN
- C21 pad 1: Net-(D12-K) -> /ESP32/BOOT
- C3 pad 1: Net-(D12-K) -> Net-(D2-K)
- C4 pad 1: Net-(D12-K) -> Net-(D2-K)
- C5 pad 1: Net-(JP1-A) -> Net-(D2-K)
- C6 pad 1: Net-(JP1-A) -> Net-(JP4-A)
- C7 pad 1: Net-(JP1-A) -> Net-(JP4-A)
- C8 pad 1: Net-(U4-RFIO) -> Net-(JP4-A)
- C9 pad 1: Net-(C9-Pad1) -> +3V3
- D1 pad 2: Net-(D1-A) -> /Power/VUSB
- D2 pad 2: Net-(D2-A) -> /Power/VUSB
- D3 pad 1: /STM32/USART1_CK -> Net-(D3-K)
- D4 pad 1: +3V3 -> Net-(D4-K)
- D4 pad 2: /STM32/SWDIO -> Net-(D4-A)
- D6 pad 1: GND -> Net-(D6-K)
- D6 pad 2: /Power/VUSB -> Net-(D6-A)
- D7 pad 2: Net-(D7-A2) -> Net-(D7-K-Pad2)
- D8 pad 1: GND -> Net-(D8-K)
- D8 pad 2: Net-(D8-A2) -> Net-(D8-A)
- FL1 pad 1: Net-(D7-A2) -> Net-(D7-K-Pad2)
- FL1 pad 2: Net-(U8-D-) -> Net-(FL1-Pad2)
- FL1 pad 3: Net-(U8-D+) -> Net-(FL1-Pad3)
- FL1 pad 4: Net-(D8-A2) -> Net-(D7-K-Pad3)
- J1 pad 1: /Power/VBAT -> Net-(Q1-D)
- J10 pad 1: GND -> Net-(J10-Pin_1)
- J10 pad 3: /STM32/SDA -> GND
- J11 pad 1: Net-(J11-Pin_1) -> GND
- J11 pad 2: /STM32/SPI2_MOSI -> Net-(J11-Pin_2)
- J11 pad 3: /STM32/SPI2_MISO -> /STM32/PA10/SDA
- J11 pad 4: /STM32/SPI2_SCK -> /STM32/PA9/SCL
- J12 pad 3: /STM32/SDA -> /STM32/PA10/SDA
- J12 pad 4: /STM32/SCL -> /STM32/PA9/SCL
- J15 pad 1: /ESP32/USB_D- -> /STM32/CP2102_~{RTS}
- J15 pad 2: /ESP32/USB_D+ -> /STM32/CP2102_~{CTS}
- J15 pad 3: GND -> /STM32/CP2102_~{DSR}
- J16 pad 1: Net-(J16-DAT2) -> Net-(J16-Pin_1)
- J16 pad 2: /ESP32/CS -> /STM32/PB15/SPI2_MOSI
- J16 pad 3: /ESP32/SDI -> /STM32/PB14/SPI2_MISO
- J16 pad 4: +3V3 -> /STM32/PB10/SPI2_SCK
- J16 pad 5: /ESP32/CLK -> /STM32/PB9/SPI2_NSS/SDI12_DIR
- J2 pad 1: Net-(Q8-D) -> SDI-12 VCC
- J2 pad 2: 0 -> GND
- J2 pad 3: unconnected-(J2-Pad3) -> Net-(J2-Pin_3)
- J3 pad 1: unconnected-(J3-Pin_1-Pad1) -> +3V3
- J3 pad 2: unconnected-(J3-Pin_2-Pad2) -> /STM32/PA13/SWDIO
- J3 pad 3: unconnected-(J3-Pin_3-Pad3) -> GND
- J3 pad 4: unconnected-(J3-Pin_4-Pad4) -> /STM32/PA14/SWDCLK
- J3 pad 5: unconnected-(J3-Pin_5-Pad5) -> GND
- J3 pad 6: unconnected-(J3-Pin_6-Pad6) -> /STM32/SWO
- J3 pad 9: unconnected-(J3-Pin_9-Pad9) -> GND
- J4 pad 1: SDI-12 VCC -> Net-(J4-In)
- J5 pad R: Net-(J4-Pin_3) -> Net-(J2-Pin_3)
- J7 pad 1: Net-(J7-In) -> GND
- J7 pad 2: GND -> Net-(J11-Pin_2)
- J8 pad 1: Net-(J8-Pin_1) -> GND
- J8 pad 2: Net-(J8-Pin_2) -> Net-(J12-Pin_2)
- J8 pad 3: GND -> /STM32/PA10/SDA
- J9 pad 2: /STM32/USART1_TX -> /STM32/PB6/USART1_TX
- J9 pad 3: /STM32/USART1_RX -> /STM32/PB7/USART1_RX
- J9 pad 5: /STM32/USART1_CTS -> /STM32/PB4/USART1_CTS
- JP1 pad 1: Net-(JP1-A) -> /Power/~{PG}
- JP1 pad 2: +3V3 -> Net-(JP1-B)
- JP10 pad 1: /STM32/USART1_RTS -> /STM32/PB13
- JP10 pad 2: Net-(JP10-B) -> /STM32/IO_INT
- JP11 pad 1: /STM32/USART1_TX -> Net-(JP11-A)
- JP11 pad 2: Net-(JP11-B) -> Net-(J2-Pin_3)
- JP12 pad 1: Net-(D12-K) -> /Power/VBAT/2
- JP12 pad 2: SDI-12 VCC -> /STM32/PA15
- JP13 pad 1: Net-(JP13-A) -> /STM32/PB5/USART1_CK
- JP13 pad 2: Net-(J4-Pin_3) -> Net-(D6-K)
- JP2 pad 2: Net-(D1-K) -> Net-(JP2-B)
- JP3 pad 1: /Power/~{PG} -> Net-(D2-K)
- JP3 pad 2: Net-(D2-K) -> SDI-12 VCC
- JP4 pad 2: unconnected-(JP4-B-Pad2) -> +3V3
- JP5 pad 1: /Power/~{PG} -> /Power/~{CHG}
- JP5 pad 2: Net-(JP5-B) -> Net-(D3-K)
- JP6 pad 1: /Power/VBAT -> /Power/~{PG}
- JP7 pad 1: +3V3 -> /Power/~{PG}
- JP7 pad 2: Net-(JP7-B) -> Net-(D4-K)
- JP8 pad 1: /STM32/USART1_RTS -> Net-(BT1-+)
- JP8 pad 2: Net-(JP8-C) -> Net-(JP8-B)
- JP9 pad 1: /STM32/USART1_RX -> /Power/SOLAR_DETECT
- L1 pad 1: Net-(U11-LX1) -> Net-(U2-LX1)
- L1 pad 2: Net-(U11-LX2) -> Net-(U2-LX2)
- Q1 pad 1: Net-(Q1-G) -> /Power/VUSB_MUX
- Q1 pad 2: GND -> Net-(D1-K)
- Q1 pad 3: /STM32/SDI12_RX -> Net-(Q1-D)
- Q2 pad 1: Net-(J10-Pin_2) -> /Power/VUSB_MUX
- Q2 pad 2: Net-(Q2-G) -> Net-(D2-K)
- Q2 pad 3: +3V3 -> Net-(BT1-+)
- Q3 pad 1: Net-(J12-Pin_2) -> /Power/VUSB_MUX
- Q3 pad 2: Net-(Q3-G) -> Net-(Q3-S)
- Q3 pad 3: +3V3 -> GND
- Q6 pad 1: Net-(J11-Pin_1) -> /STM32/I2C_PORT2_PWR
- Q6 pad 2: Net-(Q6-G) -> +3V3
- Q6 pad 3: +3V3 -> Net-(J12-Pin_2)
- Q7 pad 1: +3V3 -> /STM32/USART_PWR
- Q7 pad 2: Net-(Q7-G) -> +3V3
- Q8 pad 1: Net-(Q8-D) -> /STM32/SPI_PWR
- Q8 pad 2: Net-(Q8-G) -> +3V3
- Q8 pad 3: Net-(D11-K) -> Net-(J16-Pin_1)
- R1 pad 1: /Power/VBAT -> /Power/VUSB
- R1 pad 2: /Power/VBAT/2 -> /Power/VUSB_MUX
- R10 pad 1: Net-(JP13-A) -> Net-(JP8-B)
- R10 pad 2: Net-(D5-K) -> /Power/VBAT/2
- R11 pad 1: Net-(D5-K) -> /Power/VBAT/2
- R11 pad 2: Net-(Q1-G) -> GND
- R12 pad 1: +3V3 -> Net-(U1-ISET)
- R12 pad 2: /STM32/SDI12_RX -> GND
- R13 pad 1: GND -> Net-(U1-VDPM)
- R13 pad 2: Net-(R13-Pad2) -> Net-(Q3-S)
- R14 pad 1: Net-(C9-Pad1) -> +3V3
- R14 pad 2: Net-(J6-In) -> /STM32/IO_INT
- R15 pad 1: Net-(U4-RFIO) -> +3V3
- R15 pad 2: Net-(C9-Pad1) -> /STM32/PA10/SDA
- R16 pad 1: Net-(C9-Pad1) -> +3V3
- R16 pad 2: Net-(J7-In) -> /STM32/PA9/SCL
- R17 pad 1: /Power/VUSB -> Net-(D5-K)
- R17 pad 2: Net-(U8-VREGIN) -> Net-(Q4-G)
- R18 pad 1: +3V3 -> Net-(JP11-A)
- R18 pad 2: Net-(U8-~{RST}) -> Net-(D5-K)
- R19 pad 1: Net-(U8-TXD) -> +3V3
- R19 pad 2: /STM32/USART2_RX -> /STM32/PC0/SDI12_RX
- R2 pad 1: /Power/VBAT/2 -> +3V3
- R2 pad 2: GND -> Net-(JP1-B)
- R20 pad 1: Net-(U8-RXD) -> Net-(C12-Pad1)
- R20 pad 2: /STM32/USART2_TX -> Net-(J4-In)
- R21 pad 1: Net-(J13-CC1) -> Net-(U5-RFIO)
- R21 pad 2: GND -> Net-(C12-Pad1)
- R22 pad 1: Net-(J13-CC2) -> Net-(C12-Pad1)
- R22 pad 2: GND -> Net-(J6-In)
- R23 pad 2: Net-(D9-A) -> Net-(D6-A)
- R24 pad 1: +3V3 -> /STM32/I2C_PORT1_PWR
- R24 pad 2: Net-(D10-A) -> GND
- R26 pad 1: GND -> /STM32/USART_PWR
- R26 pad 2: Net-(U11-FB) -> GND
- R27 pad 1: Net-(U9-IO8) -> Net-(J10-Pin_2)
- R27 pad 2: +3V3 -> Net-(J10-Pin_1)
- R28 pad 1: Net-(U9-IO2) -> Net-(U10-VREGIN)
- R29 pad 1: Net-(U9-IO18) -> /Power/VUSB
- R29 pad 2: /ESP32/USB_D- -> Net-(U10-VREGIN)
- R3 pad 1: Net-(JP6-B) -> +3V3
- R3 pad 2: Net-(D1-A) -> Net-(JP2-B)
- R30 pad 1: Net-(U9-IO19) -> Net-(U10-TXD)
- R30 pad 2: /ESP32/USB_D+ -> /STM32/PA3/USART2_RX
- R31 pad 1: /ESP32/ESP32_EN -> Net-(F1-Pad1)
- R31 pad 2: /ESP32/EN -> /Power/VUSB
- R34 pad 1: Net-(Q6-G) -> Net-(J14-CC1)
- R35 pad 1: Net-(Q2-G) -> Net-(J14-CC2)
- R36 pad 1: Net-(Q3-G) -> +3V3
- R36 pad 2: GND -> Net-(D8-A)
- R37 pad 1: Net-(Q7-G) -> +3V3
- R37 pad 2: GND -> Net-(D9-A)
- R38 pad 1: +3V3 -> /STM32/SPI_PWR
- R38 pad 2: /STM32/SDA -> GND
- R39 pad 1: +3V3 -> Net-(U11-IO8)
- R39 pad 2: /STM32/SCL -> +3V3
- R4 pad 1: Net-(JP6-B) -> /Power/VUSB_MUX
- R4 pad 2: Net-(D2-A) -> GND
- R40 pad 1: Net-(Q8-G) -> Net-(U11-IO2)
- R40 pad 2: GND -> +3V3
- R41 pad 1: Net-(Q8-G) -> Net-(U11-IO18)
- R41 pad 2: /Power/VUSB -> /ESP32/USB_D-
- R42 pad 1: Net-(Q9-G) -> Net-(U11-IO19)
- R42 pad 2: /Power/VUSB -> /ESP32/USB_D+
- R43 pad 1: Net-(Q9-G) -> /STM32/PA0
- R43 pad 2: GND -> /ESP32/EN
- R44 pad 1: Net-(Q10-G) -> Net-(FL1-Pad2)
- R44 pad 2: /Power/VUSB -> Net-(U10-D-)
- R45 pad 1: Net-(Q10-G) -> Net-(FL1-Pad3)
- R45 pad 2: GND -> Net-(U10-D+)
- R5 pad 1: Net-(JP4-A) -> Net-(BT1-+)
- R5 pad 2: /Power/VBAT/2 -> Net-(D3-A)
- R6 pad 1: /Power/VBAT/2 -> Net-(BT1-+)
- R6 pad 2: 0 -> Net-(D4-A)
- R7 pad 1: Net-(U1-VDPM) -> +3V3
- R7 pad 2: Net-(Q9-D) -> Net-(JP9-B)
- R8 pad 1: Net-(U1-ISET) -> Net-(U2-CFG1)
- R8 pad 2: 0 -> GND
- R9 pad 1: +3V3 -> Net-(U1-VTSB)
- R9 pad 2: Net-(D3-A) -> Net-(U1-TS)
- RN1 pad 1: Net-(J16-DAT1) -> Net-(J19-DAT1)
- RN1 pad 4: Net-(J16-DAT2) -> Net-(J19-DAT2)
- SW3 pad 1: /STM32/RST -> GND
- SW3 pad 2: GND -> /ESP32/EN
- SW4 pad 1: /STM32/PB13 -> GND
- SW4 pad 2: Net-(R13-Pad2) -> /ESP32/BOOT
- TH1 pad 2: 0 -> GND
- TP1 pad 1: Net-(D11-K) -> Net-(D1-K)
- U1 pad 1: Net-(D11-K) -> Net-(D1-K)
- U1 pad 10: Net-(JP6-B) -> Net-(BT1-+)
- U1 pad 11: 0 -> GND
- U1 pad 3: 0 -> GND
- U1 pad 7: Net-(JP5-B) -> Net-(JP6-B)
- U10 pad 1: unconnected-(U10-~{INT}-Pad1) -> /STM32/CP2102_~{RI}
- U10 pad 11: unconnected-(U10-P07-Pad11) -> /STM32/CP2102_~{WAKEUP}
- U10 pad 12: GND -> /STM32/CP2102_RS485
- U10 pad 13: unconnected-(U10-P10-Pad13) -> Net-(D9-K)
- U10 pad 14: unconnected-(U10-P11-Pad14) -> Net-(D8-K)
- U10 pad 15: unconnected-(U10-P12-Pad15) -> /STM32/CP2102_~{SUSPEND}
- U10 pad 17: unconnected-(U10-P14-Pad17) -> /STM32/CP2102_SUSPEND
- U10 pad 18: unconnected-(U10-P15-Pad18) -> /STM32/CP2102_~{CTS}
- U10 pad 19: unconnected-(U10-P16-Pad19) -> /STM32/CP2102_~{RTS}
- U10 pad 20: unconnected-(U10-P17-Pad20) -> Net-(U10-RXD)
- U10 pad 21: GND -> Net-(U10-TXD)
- U10 pad 22: /STM32/SCL -> /STM32/CP2102_~{DSR}
- U10 pad 23: /STM32/SDA -> Net-(U10-~{DTR})
- U10 pad 24: +3V3 -> /STM32/CP2102_~{DCD}
- U10 pad 3: GND -> Net-(U10-D+)
- U10 pad 4: unconnected-(U10-P00-Pad4) -> Net-(U10-D-)
- U10 pad 5: unconnected-(U10-P01-Pad5) -> +3V3
- U10 pad 6: unconnected-(U10-P02-Pad6) -> +3V3
- U10 pad 7: unconnected-(U10-P03-Pad7) -> Net-(U10-VREGIN)
- U10 pad 8: unconnected-(U10-P04-Pad8) -> Net-(U10-VBUS)
- U10 pad 9: unconnected-(U10-P05-Pad9) -> Net-(U10-~{RST})
- U11 pad 1: Net-(JP1-A) -> +3V3
- U11 pad 2: Net-(U11-LX2) -> /ESP32/EN
- U11 pad 3: Net-(U11-LX1) -> /ESP32/CLK
- U11 pad 4: Net-(D12-K) -> /ESP32/SDO
- U11 pad 5: unconnected-(U11-EN-Pad5) -> /ESP32/SDI
- U11 pad 6: unconnected-(U11-MODE-Pad6) -> /ESP32/CS
- U11 pad 7: GND -> Net-(U11-IO8)
- U11 pad 8: Net-(U11-FB) -> /ESP32/BOOT
- U4 pad 1: +3V3 -> /STM32/PB9/SPI2_NSS/SDI12_DIR
- U4 pad 2: GND -> /STM32/PC1/SDI12_TX
- U4 pad 3: /STM32/SWDIO -> GND
- U4 pad 4: /STM32/SWDCLK -> Net-(Q4-G)
- U4 pad 5: /STM32/SPI2_MOSI -> SDI-12 VCC
- U5 pad 1: unconnected-(U5-NC-Pad1) -> +3V3
- U5 pad 2: unconnected-(U5-A1-Pad2) -> GND
- U5 pad 3: unconnected-(U5-A2-Pad3) -> /STM32/PA13/SWDIO
- U5 pad 4: GND -> /STM32/PA14/SWDCLK
- U5 pad 5: /STM32/SDA -> /STM32/PB15/SPI2_MOSI
- U5 pad 6: /STM32/SCL -> /STM32/PA15
- U5 pad 7: unconnected-(U5-WP-Pad7) -> /STM32/PB4/USART1_CTS
- U5 pad 8: +3V3 -> /STM32/PB3
- U6 pad 1: Net-(JP9-B) -> unconnected-(U6-NC-Pad1)
- U6 pad 2: Net-(JP10-B) -> unconnected-(U6-A1-Pad2)
- U6 pad 3: Net-(JP10-B) -> unconnected-(U6-A2-Pad3)
- U6 pad 4: Net-(JP11-B) -> GND
- U6 pad 5: GND -> /STM32/PA10/SDA
- U6 pad 6: Net-(J8-Pin_1) -> /STM32/PA9/SCL
- U6 pad 7: Net-(J8-Pin_2) -> unconnected-(U6-WP-Pad7)
- U6 pad 8: Net-(JP7-B) -> +3V3
- U7 pad 1: unconnected-(U7-NC-Pad1) -> Net-(JP15-B)
- U7 pad 2: +3V3 -> Net-(JP16-B)
- U7 pad 3: GND -> Net-(JP17-A)
- U7 pad 4: GND -> Net-(JP19-B)
- U7 pad 5: /STM32/SDA -> GND
- U7 pad 6: /STM32/SCL -> Net-(J10-Pin_1)
- U7 pad 7: unconnected-(U7-WP-Pad7) -> Net-(J10-Pin_2)
- U7 pad 8: +3V3 -> Net-(J9-Pin_1)
- U8 pad 2: GND -> +3V3
- U8 pad 3: Net-(U8-D+) -> GND
- U8 pad 4: Net-(U8-D-) -> GND
- U8 pad 5: +3V3 -> /STM32/PA10/SDA
- U8 pad 6: +3V3 -> /STM32/PA9/SCL
- U8 pad 7: Net-(U8-VREGIN) -> unconnected-(U8-WP-Pad7)
- U8 pad 8: /Power/VUSB -> +3V3
- U9 pad 1: +3V3 -> /STM32/IO_INT
- U9 pad 10: /ESP32/CD -> /STM32/SPI_PWR
- U9 pad 11: /ESP32/RX -> /Power/TPS631000_EN
- U9 pad 12: /ESP32/TX -> GND
- U9 pad 13: Net-(U9-IO18) -> /Power/TPS631000_MODE
- U9 pad 14: Net-(U9-IO19) -> /Power/SOLAR_DETECT
- U9 pad 15: /ESP32/WAKEUP -> /STM32/IO_P12
- U9 pad 16: Net-(U9-IO2) -> /STM32/IO_P13
- U9 pad 17: /STM32/SCL -> /STM32/IO_P14
- U9 pad 18: /STM32/SDA -> /STM32/IO_P15
- U9 pad 2: /ESP32/EN -> GND
- U9 pad 3: /ESP32/CLK -> GND
- U9 pad 4: /ESP32/SDO -> /ESP32/WAKEUP
- U9 pad 5: /ESP32/SDI -> /Power/~{CHG}
- U9 pad 6: /ESP32/CS -> /Power/~{PG}
- U9 pad 7: Net-(U9-IO8) -> /STM32/USART_PWR
- U9 pad 8: /ESP32/BOOT -> /STM32/I2C_PORT1_PWR
- U9 pad 9: GND -> /STM32/I2C_PORT2_PWR
Routing:
- net (no net): track 375.0 -> 0.00 mm, vias 1 -> 0
- net +3V3: track 285.8 -> 0.00 mm, vias 17 -> 12
- net GND: track 172.4 -> 0.00 mm, vias 14 -> 17
- net /STM32/SDA: track 93.2 -> 0.00 mm, vias 2 -> 0
- net /STM32/SCL: track 90.9 -> 0.00 mm, vias 4 -> 0
- net /ESP32/EN: track 70.1 -> 0.00 mm, vias 2 -> 3
- net /STM32/RST: track 66.4 -> 0.00 mm
- net /ESP32/BOOT: track 60.9 -> 0.00 mm, vias 2 -> 0
- net /STM32/SDI12_RX: track 59.0 -> 0.00 mm
- net /Power/VBAT: track 49.6 -> 0.00 mm, vias 2 -> 0
- net /ESP32/ESP32_EN: track 47.2 -> 0.00 mm
- net /ESP32/WAKEUP: track 44.1 -> 0.00 mm
- net /ESP32/CD: track 35.1 -> 0.00 mm
- net Net-(J7-In): track 34.6 -> 0.00 mm, vias 2 -> 0
- net /ESP32/CS: track 26.7 -> 0.00 mm
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Other:
- board size 151 x 103.2 mm -> 100 x 50 mm

Commit message: PCB layout with silkscreen annotations
Parts:
- removed the J10 at (-36.5, 98.0)
- removed the J13 at (121.0, 186.5)
- removed J15: Conn_02x05_Top_Bottom, Connector_PinHeader_2.54mm:PinHeader_2x05_P2.54mm_Vertical
- removed JP15, JP16, JP17, JP18, JP19: SolderJumper_2_Open, Jumper:SolderJumper-2_P1.3mm_Open_RoundedPad1.0x1.5mm
- removed the JP6 at (43.0, -19.8)
- removed the JP8 at (75.8, -27.3)
- removed the R27 at (-27.5, 108.1)
- removed U7: SN65HVD11HD, Package_SO:SOIC-8_3.9x4.9mm_P1.27mm
- added J14: Conn_02x04_Odd_Even, Connector_PinHeader_2.54mm:PinHeader_2x04_P2.54mm_Vertical, F.Cu at (166.3, 135.7)
- added J17: Conn_02x04_Odd_Even, Connector_PinHeader_2.54mm:PinHeader_2x04_P2.54mm_Vertical, F.Cu at (166.2, 123.2)
- added JP7: SolderJumper_2_Open, Jumper:SolderJumper-2_P1.3mm_Open_RoundedPad1.0x1.5mm, B.Cu at (111.5, 139.7)
- J12: renamed from J9; value Conn_01x06_Pin -> Conn_02x04_Odd_Even
- J3: footprint Soil Power Sensor:ARM10_DEBUG -> Soil Power Sensor:SAMTEC_FTSH-105-01-X-DV-K-P
- J4: footprint Connector_Coaxial:SMA_Molex_73251-1153_EdgeMount_Horizontal -> Connector_Coaxial:SMA_Samtec_SMA-J-P-H-ST-EM1_EdgeMount
- JP1, JP2, JP5: moved to B.Cu
- JP10: renamed from JP11; moved to B.Cu
- JP11: renamed from JP12; moved to B.Cu
- JP12: renamed from JP13; moved to B.Cu
- JP13: renamed from JP14; moved to B.Cu
- JP6: renamed from JP7; moved to B.Cu
- JP9: renamed from JP10; moved to B.Cu
- moved Q4 281.9 mm to (145.8, 112.4), turned to 0 degrees
- moved R19 278.0 mm to (148.5, 112.4), turned to 90 degrees
- moved D5 274.6 mm to (147.0, 116.5)
- moved R17 273.9 mm to (149.5, 116.2), turned to 90 degrees
- moved R18 273.9 mm to (144.5, 116.2), turned to -90 degrees
- moved J5 271.1 mm to (137.8, 109.8), turned to 0 degrees
- moved JP10 265.0 mm to (142.0, 112.5)
- moved U4 261.0 mm to (151.5, 112.5)
- moved J19 258.2 mm to (138.1, 143.2), turned to 180 degrees
- moved R44 257.6 mm to (142.6, 144.6), turned to 180 degrees
- moved Q5 254.6 mm to (112.8, 108.2), turned to 180 degrees
- moved R46 253.3 mm to (142.6, 143.1), turned to 180 degrees
- moved R45 250.8 mm to (142.6, 141.6), turned to 180 degrees
- moved R24 248.1 mm to (115.5, 108.2), turned to 90 degrees
- moved U11 248.0 mm to (154.1, 146.2), turned to 180 degrees
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- renumbered J11 to J10, J12 to J11, J16 to J13, J14 to J16, J17 to J19, J18 to J20, J19 to J21, JP9 to JP8, Q8 to Q7, Q7 to Q8, R38 to R27, R26 to R28, R28 to R29, R29 to R30, R30 to R31, R31 to R32, R32 to R33, R46 to R34, R33 to R35, R34 to R36, R47 to R37, R35 to R38, R44 to R39, R45 to R40, R36 to R41, R37 to R42, R39 to R43, R40 to R44, R41 to R45, R42 to R46, R43 to R47
Connections:
- net Net-(J9-Pin_1) renamed /STM32/USART1_VCC
- FL1 pad 1: Net-(D7-K-Pad2) -> Net-(D7-K-Pad3)
- FL1 pad 4: Net-(D7-K-Pad3) -> Net-(D7-K-Pad2)
- J12 pad 2: /STM32/PB6/USART1_TX -> /STM32/PB4/USART1_CTS
- J12 pad 3: /STM32/PB7/USART1_RX -> /STM32/PB6/USART1_TX
- J12 pad 4: GND -> /STM32/USART1_RTS
- J12 pad 5: /STM32/PB4/USART1_CTS -> /STM32/PB7/USART1_RX
- J12 pad 6: /STM32/USART1_RTS -> /STM32/PB5/USART1_CK
- U1 pad 7: Net-(JP6-B) -> /Power/~{PG}
Routing:
- net +3V3: track 0.00 -> 357.0 mm, vias 12 -> 14
- net /STM32/PA9/SCL: track 0.00 -> 171.1 mm, vias 6 -> 8
- net /STM32/PA10/SDA: track 0.00 -> 165.7 mm, vias 2 -> 7
- net GND: track 0.00 -> 154.4 mm, vias 17 -> 123
- net /Power/VBAT/2: track 0.00 -> 87.5 mm, vias 0 -> 1
- net /Power/VUSB: track 0.00 -> 85.9 mm, vias 0 -> 6
- net /STM32/PB9/SPI2_NSS/SDI12_DIR: track 0.00 -> 85.2 mm, vias 0 -> 4
- net /STM32/PC0/SDI12_RX: track 0.00 -> 79.0 mm, vias 0 -> 2
- net /STM32/RST: track 0.00 -> 77.1 mm, vias 0 -> 4
- net /STM32/PC1/SDI12_TX: track 0.00 -> 75.9 mm, vias 0 -> 2
- net /STM32/PB13: track 0.00 -> 71.4 mm, vias 0 -> 3
- net /Power/~{CHG}: track 0.00 -> 66.0 mm, vias 1 -> 2
- net /Power/~{PG}: track 0.00 -> 65.4 mm, vias 0 -> 2
- net /Power/SOLAR_DETECT: track 0.00 -> 58.8 mm, vias 0 -> 3
- net /STM32/USART_PWR: track 0.00 -> 57.4 mm, vias 0 -> 4
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Other:
- board text added: "(only on during first charge cycle)"
- board text added: "103AT NTC Thermistor"
- board text added: "3.3V ENABLE"
- board text added: "3.3V IO_P13 IO_P15 IO_P17"
- board text added: "3.3V MOSI MISO SCK NSS GND"
- board text added: "3.3V PB3 (USART1_RTS/SWO) PC0/SDI12_RX B9/SDI12_DIR"
- board text added: "3.3V SDI-12 VCC V_{BAT} | V_{USB}"
- board text added: "3.3V TX RX GND"
- board text added: "CTS RTS CK GND"
- board text added: "Charge LED"
- board text added: "Data GND VCC"
- board text added: "ESP32 CDC"
- board text added: "ESP32 UART"
- board text added: "Enable V_{BAT} resistor divider TP2."
- board text added: "GND 3.3V SDA SCL"
- board text added: "GND D- D+"
- board text added: "GND RX TX"
- board text added: "I2C Port 1"
- board text added: "I2C Port 2"
- board text added: "IO expander ~{INT}"
- board text added: "IO_P12 IO_P14 IO_P16 GND"
- board text added: "JP3: 3.3V SDI-12 VCC V_{BAT} | V_{USB}"
- board text added: "JP4: 3.3V ENABLE"
- board text added: "Li-Ion Battery"
- board text added: "PA15 (V_{BAT}/2) PB13 (SW2, IO_~{INT}) PC1/SDI12_TX GND"
- board text added: "PB2 redirect >1-2: USART1_RTS 2-3: SWO (SWD/JTAG)"
- board text added: "Power Good LED"
- board text added: "SCL SDA 3.3V GND"
- board text added: "SDI-12 3.5mm Tip: VCC Ring: Data Shaft: GND"
- board text added: "SDI-12 transceiver select. >1-2: External transceiver 2-3: Internal transceiver"
- board text added: "SPI"
- board text added: "Solar Input V_{OC_Max}<= 18 V Typical: V_{OC}=6 V"
- board text added: "Solar input detect (IO_P11)"
- board text added: "UART RXT"
- board text added: "UART TXT"
- board text added: "USART1"
- board text added: "User LED (PB5)"
- board text added: "V_{BAT}/2 analog input (PA15)"
- board text added: "~{PG} (JP1) ~{CHG} (JP2) external pullups."
- board text removed: "BOOT"
- board text removed: "D+"
- board text removed: "D-"
- board text removed: "DTR"
- board text removed: "Data"
- board text removed: "GND"
- board text removed: "I2C"
- board text removed: "RST"
- board text removed: "RTS"
- board text removed: "RX"
- board text removed: "SDI12"
- board text removed: "TX"
- board text removed: "VCC"

Commit message: finishing touches and fabrication output
Parts:
- removed J10: Conn_01x04_Pin, Connector_PinSocket_2.54mm:PinSocket_1x04_P2.54mm_Vertical
- removed the J20 at (142.1, 138.7)
- added J2: ~, Connector_JST:JST_PH_S2B-PH-SM4-TB_1x02-1MP_P2.00mm_Horizontal, F.Cu at (113.5, 144.7)
- BT1: footprint Connector_JST:JST_PH_S2B-PH-K_1x02_P2.00mm_Horizontal -> Connector_PinHeader_2.54mm:PinHeader_1x02_P2.54mm_Vertical
- C10, C11, C12, C13, C15, C16, C18, C19, C21, C3, C6: value 0.1uF -> 100nF
- C5, C8: footprint Capacitor_SMD:C_0603_1608Metric -> Capacitor_SMD:C_0805_2012Metric
- D1, D2: value RB521S-40 -> RB160M-30; footprint Diode_SMD:D_SOD-523 -> Diode_SMD:D_SOD-123
- D5: value BZX84Cxx -> BZX84C7V5
- D7: value SP0503BAHT -> SP0503BAHTG
- J1: footprint Connector_BarrelJack:BarrelJack_Horizontal -> Connector_BarrelJack:BarrelJack_Wuerth_694106106102_2.0x5.5mm
- J11: value Conn_01x04_Pin -> Conn_02x04_Odd_Even; footprint Connector_PinSocket_2.54mm:PinSocket_1x04_P2.54mm_Vertical -> Connector_PinHeader_2.54mm:PinHeader_2x04_P2.54mm_Vertical
- J13: value Conn_01x04_Pin -> Conn_01x06_Pin
- J16: renamed from J17; value Conn_02x04_Odd_Even -> Conn_02x05_Odd_Even; footprint Connector_PinHeader_2.54mm:PinHeader_2x04_P2.54mm_Vertical -> Connector_PinHeader_2.54mm:PinHeader_2x05_P2.54mm_Vertical
- J17: renamed from J16; footprint Connector_USB:USB_C_Receptacle_GCT_USB4110 -> Connector_USB:USB_C_Receptacle_G-Switch_GT-USB-7010ASV
- J19: value Conn_01x03 -> Conn_02x04_Odd_Even; footprint Connector_PinHeader_2.54mm:PinHeader_1x03_P2.54mm_Vertical -> Connector_PinHeader_2.54mm:PinHeader_2x04_P2.54mm_Vertical
- J6: renamed from J5; footprint Connector_Audio:Jack_3.5mm_CUI_SJ-3523-SMT_Horizontal -> Soil Power Sensor:Jack_3.5mm_PJ313D_Horizontal
- JP12: footprint Jumper:SolderJumper-2_P1.3mm_Bridged_RoundedPad1.0x1.5mm -> Jumper:SolderJumper-2_P1.3mm_Open_RoundedPad1.0x1.5mm
- JP3: value SolderJumper_3_Open -> SolderJumper_3_Bridged12
- JP5, JP6, JP7: value SolderJumper_2_Open -> SolderJumper_2_Bridged
- JP8: moved to B.Cu
- R10: renamed from R12; value 680 -> 680R
- R17, R18: value 510 -> 510R
- R20, R21, R22, R29, R30, R32, R39, R40, R45, R46: value 0 -> 0R
- R31, R33: value 20 -> 20R
- SW1: value RST -> STM32_RST; footprint Button_Switch_SMD:SW_Push_1P1T_NO_CK_KSC7xxJ -> Button_Switch_SMD:SW_Push_1P1T_XKB_TS-1187A
- SW2: value BOOT/USER -> STM32_BOOT/USER; footprint Button_Switch_SMD:SW_Push_1P1T_NO_CK_KSC7xxJ -> Button_Switch_SMD:SW_Push_1P1T_XKB_TS-1187A
- SW3: value EN -> ESP32_EN; footprint Button_Switch_SMD:SW_Push_1P1T_NO_CK_KSC7xxJ -> Button_Switch_SMD:SW_Push_1P1T_XKB_TS-1187A
- SW4: value BOOT -> ESP32_BOOT; footprint Button_Switch_SMD:SW_Push_1P1T_NO_CK_KSC7xxJ -> Button_Switch_SMD:SW_Push_1P1T_XKB_TS-1187A
- U11: footprint Soil Power Sensor:MODULE_ESP32-C3-WROOM-02-N4 -> RF_Module:ESP32-C3-WROOM-02
- U6, U8: footprint Soil Power Sensor:SOP127P505X155-8N -> Package_SO:SSOP-8_3.9x5.05mm_P1.27mm
- moved C21 20.6 mm to (165.5, 147.4), turned to 0 degrees
- moved JP7 7.10 mm to (118.0, 136.8), turned to -90 degrees
- moved J19 7.05 mm to (138.2, 136.2), turned to 0 degrees
- moved J6 6.71 mm to (137.4, 103.1), turned to -90 degrees
- moved J1 5.67 mm to (108.6, 126.1), turned to -90 degrees
- moved BT1 5.49 mm to (112.1, 137.8), turned to 90 degrees
- moved JP5 4.76 mm to (105.7, 133.1)
- moved JP6 4.69 mm to (105.7, 135.6)
- moved R12 4.12 mm to (118.0, 139.0)
- moved R13 4.12 mm to (118.0, 137.5)
- moved R2 3.94 mm to (118.0, 131.0)
- moved R7 3.94 mm to (116.5, 131.0)
- moved R5 3.63 mm to (107.2, 133.9)
- moved R3 3.51 mm to (119.5, 131.0), turned to -90 degrees
- moved TH1 3.38 mm to (120.2, 143.1)
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- renumbered J21 to J20, J2 to J3, J3 to J4, J4 to J5, J6 to J7, J7 to J8, J8 to J9, R13 to R11, R10 to R12, R11 to R13, R44 to R43, R43 to R44
Connections:
- J11 pad 2: Net-(J11-Pin_2) -> GND
- J11 pad 3: /STM32/PA10/SDA -> Net-(J11-Pin_3)
- J11 pad 4: /STM32/PA9/SCL -> Net-(J11-Pin_4)
- J16 pad 2: /STM32/IO_P12 -> /STM32/IO_P10
- J16 pad 3: /STM32/IO_P13 -> /STM32/IO_P11
- J16 pad 4: /STM32/IO_P14 -> /STM32/IO_P12
- J16 pad 5: /STM32/IO_P15 -> /STM32/IO_P13
- J16 pad 6: /STM32/IO_P16 -> /STM32/IO_P14
- J16 pad 7: /STM32/IO_P17 -> /STM32/IO_P15
- J16 pad 8: GND -> /STM32/IO_P16
- J19 pad 1: /ESP32/USB_D+ -> +3V3
- J19 pad 2: /ESP32/USB_D- -> +3V3
- J19 pad 3: GND -> /ESP32/USB_D-
- J8 pad 2: Net-(J10-Pin_2) -> Net-(J11-Pin_3)
- J9 pad 2: Net-(J11-Pin_2) -> Net-(J11-Pin_4)
- Q5 pad 3: Net-(J10-Pin_2) -> Net-(J11-Pin_3)
- Q6 pad 3: Net-(J11-Pin_2) -> Net-(J11-Pin_4)
- R39 pad 1: Net-(FL1-Pad2) -> Net-(FL1-Pad3)
- R40 pad 1: Net-(FL1-Pad3) -> Net-(FL1-Pad2)
- U2 pad 1: /Power/TPS631000_EN -> Net-(D2-K)
- U2 pad 2: /Power/TPS631000_MODE -> Net-(D2-K)
- U9 pad 11: /Power/TPS631000_EN -> /Power/SOLAR_DETECT
- U9 pad 13: /Power/TPS631000_MODE -> /STM32/IO_P10
- U9 pad 14: /Power/SOLAR_DETECT -> /STM32/IO_P11
Routing:
- net GND: track 154.4 -> 186.6 mm, vias 123 -> 92
- net /Power/TPS631000_MODE: track 31.3 -> 0.00 mm, vias 2 -> 0
- net /Power/TPS631000_EN: track 23.0 -> 0.00 mm, vias 2 -> 0
- net /STM32/IO_P11: track 0.00 -> 15.9 mm
- net Net-(J11-Pin_4): track 0.00 -> 13.6 mm
- net Net-(J11-Pin_3): track 0.00 -> 11.1 mm
- net /Power/VBAT/2: track 87.5 -> 77.7 mm
- net Net-(J11-Pin_2): track 9.67 -> 0.00 mm
- net /STM32/IO_P10: track 0.00 -> 9.14 mm
- net Net-(J10-Pin_2): track 8.78 -> 0.00 mm
- net Net-(Q1-D): track 4.97 -> 12.9 mm
- net Net-(J3-Pin_3): track 11.2 -> 18.6 mm
- net /STM32/PA9/SCL: track 171.1 -> 165.1 mm
- net Net-(BT1-+): track 55.1 -> 60.0 mm
- net /STM32/USART_PWR: track 57.4 -> 52.6 mm, vias 4 -> 6
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Other:
- board text added: "- +"
- board text added: "3.3V D- D+ GND"
- board text added: "3.3V IO_P11 IO_P13 IO_P15 IO_P17"
- board text added: "3.3V RX TX GND"
- board text added: "3.3V SDI-12 VCC --> V_{BAT} | V_{USB}"
- board text added: "Charge"
- board text added: "ESP32 USB CDC"
- board text added: "Enable V_{BAT}/2 resistor divider TP2"
- board text added: "IO_P10 IO_P12 IO_P14 IO_P16 GND"
- board text added: "Power"
- board text added: "RXT"
- board text added: "Solar detect (IO_P07)"
- board text added: "TXT"
- board text added: "~{PG} (JP1) ~{CHG} (JP2) external pullups"
- board text removed: "(only on during first charge cycle)"
- board text removed: "3.3V IO_P13 IO_P15 IO_P17"
- board text removed: "3.3V SDI-12 VCC V_{BAT} | V_{USB}"
- board text removed: "Charge LED"
- board text removed: "ESP32 CDC"
- board text removed: "Enable V_{BAT} resistor divider TP2."
- board text removed: "GND D- D+"
- board text removed: "GND RX TX"
- board text removed: "IO_P12 IO_P14 IO_P16 GND"
- board text removed: "Power Good LED"
- board text removed: "Solar input detect (IO_P11)"
- board text removed: "UART RXT"
- board text removed: "UART TXT"
- board text removed: "~{PG} (JP1) ~{CHG} (JP2) external pullups."
