File: hardware/Soil_Power_Sensor_5.kicad_sch (KiCad schematic)
At the start: 8 parts, among them J10 Conn_01x03, U7 SN65HVD11HD

Commit message: 3.1.0 tidy layout, single header
Parts:
- renumbered J10 to J16, R26 to R47, U7 to U10
Changed lines of the file:
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@@
 	(generator_version "9.0")
 	(paper "A4")
+	(title_block
+		(date "2026-04-06")
+		(rev "3.1.0")
+	)
 	(rectangle
 		(start 13.97 13.97)
@@
 		(on_board no)
 		(dnp yes)
-		(property "Reference" "R26"
+		(property "Reference" "R47"
 			(at 62.23 43.18 0)
 			(effects
@@
 			(project "Soil Power Sensor"
 				(path "/5300ec4d-4648-40a1-8d89-4fa6b3bf32a3/43a883bb-5678-46a3-a756-4c64cbfd0ddc/e11527b4-1666-4b88-a9f5-c91ece62b2a8"
-					(reference "R26")
+					(reference "R47")
 					(unit 1)
 				)
@@
 		(on_board no)
 		(dnp yes)
-		(property "Reference" "J10"
+		(property "Reference" "J16"
 			(at 66.548 30.734 0)
 			(effects
@@
 			(project "Soil Power Sensor"
 				(path "/5300ec4d-4648-40a1-8d89-4fa6b3bf32a3/43a883bb-5678-46a3-a756-4c64cbfd0ddc/e11527b4-1666-4b88-a9f5-c91ece62b2a8"
-					(reference "J10")
+					(reference "J16")
 					(unit 1)
 				)
@@
 		(dnp no)
 		(fields_autoplaced yes)
-		(property "Reference" "#PWR056"
+		(property "Reference" "#PWR091"
 			(at 50.8 57.15 0)
 			(effects
@@
 			(project "Soil Power Sensor"
 				(path "/5300ec4d-4648-40a1-8d89-4fa6b3bf32a3/43a883bb-5678-46a3-a756-4c64cbfd0ddc/e11527b4-1666-4b88-a9f5-c91ece62b2a8"
-					(reference "#PWR056")
+					(reference "#PWR091")
 					(unit 1)
 				)
@@
 		(dnp no)
 		(fields_autoplaced yes)
-		(property "Reference" "#PWR052"
+		(property "Reference" "#PWR090"
 			(at 69.85 48.26 0)
 			(effects
@@
 			(project "Soil Power Sensor"
 				(path "/5300ec4d-4648-40a1-8d89-4fa6b3bf32a3/43a883bb-5678-46a3-a756-4c64cbfd0ddc/e11527b4-1666-4b88-a9f5-c91ece62b2a8"
-					(reference "#PWR052")
+					(reference "#PWR090")
 					(unit 1)
 				)
@@
 		(on_board yes)
 		(dnp no)
-		(property "Reference" "#FLG04"
+		(property "Reference" "#FLG06"
 			(at 45.72 20.955 0)
 			(effects
@@
 			(project "Soil Power Sensor"
 				(path "/5300ec4d-4648-40a1-8d89-4fa6b3bf32a3/43a883bb-5678-46a3-a756-4c64cbfd0ddc/e11527b4-1666-4b88-a9f5-c91ece62b2a8"
-					(reference "#FLG04")
+					(reference "#FLG06")
 					(unit 1)
 				)
@@
 		(dnp yes)
 		(fields_autoplaced yes)
-		(property "Reference" "U7"
+		(property "Reference" "U10"
 			(at 52.9433 22.86 0)
 			(effects
@@
 			(project "Soil Power Sensor"
 				(path "/5300ec4d-4648-40a1-8d89-4fa6b3bf32a3/43a883bb-5678-46a3-a756-4c64cbfd0ddc/e11527b4-1666-4b88-a9f5-c91ece62b2a8"
-					(reference "U7")
+					(reference "U10")
 					(unit 1)
 				)
