File: extra/analog_multiplexer/Analog Multiplexer.kicad_sch (KiCad schematic)
At the start: 13 parts, among them J1 Conn_01x05_Socket, J2 Conn_01x05_Socket, J3 Conn_01x05_Socket, J4 Conn_01x05_Socket, J5 Conn_01x05_Socket, J6 Conn_01x04_Socket, U1 TLV1117-33, U4 ADG729, U5 ADG729

Commit message: Generated production files
Other:
- company: (none) -> jLab
- title: (none) -> Analog Multiplexer
Changed lines of the file:
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@@
 	(generator_version "9.0")
 	(paper "A4")
+	(title_block
+		(title "Analog Multiplexer")
+		(date "2025-09-30")
+		(rev "v1")
+		(company "jLab")
+	)
 	(text "Set A0 to 1 and A1 to 0\nI2C Value is 0x45"
 		(exclude_from_sim no)
